Commit message: Fix error

File: democar_gazebo/urdf/depth_camera.xacro (robot description, xacro)
@@ -15,5 +15,5 @@
             <origin xyz="0 0 0" rpy="0 0 0"/>
             <geometry>
-                <mesh filename="$(find rlcar_gazebo)/meshes/depth435.stl" scale="0.001 0.001 0.001"/>
+                <mesh filename="$(find democar_gazebo)/meshes/depth435.stl" scale="0.001 0.001 0.001"/>
             </geometry>
             <material name="silver"/>
@@ -22,5 +22,5 @@
             <origin xyz="0 0 0" rpy="0 0 0"/>
             <geometry>
-                <mesh filename="$(find rlcar_gazebo)/meshes/depth435.stl" scale="0.001 0.001 0.001"/>
+                <mesh filename="$(find democar_gazebo)/meshes/depth435.stl" scale="0.001 0.001 0.001"/>
             </geometry>
         </collision>
